File: Hardware/SparkFun_Qwiic_Micro_SAMD21E.brd (EAGLE design)
At the start: 25.4 x 25.4 mm, 80 parts, among them Q1 3.1A/30V/105mΩ, U1 3.3V, U2 W25Q32FV, U3 ATSAMD21E18A-U

Commit message: Updates dimensions...
Parts:
- moved FRAME1 11.0 mm to (-13.7, -20.1)
- moved J2 0.25 mm to (24.1, 6.35)
Changed lines of the file:
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@@
 <layer number="37" name="tTest" color="7" fill="1" visible="no" active="yes"/>
 <layer number="38" name="bTest" color="7" fill="1" visible="no" active="yes"/>
-<layer number="39" name="tKeepout" color="4" fill="11" visible="yes" active="yes"/>
+<layer number="39" name="tKeepout" color="4" fill="11" visible="no" active="yes"/>
 <layer number="40" name="bKeepout" color="1" fill="11" visible="no" active="yes"/>
 <layer number="41" name="tRestrict" color="4" fill="10" visible="no" active="yes"/>
@@
 <wire x1="0" y1="25.4" x2="0" y2="0" width="0.2032" layer="20"/>
 <text x="7.9248" y="0.2794" size="0.8128" layer="16" font="vector" ratio="15" rot="MR0">V10</text>
-<text x="35.687" y="-9.652" size="1.778" layer="51" font="vector" align="bottom-right">Michelle Shorter</text>
-<text x="1.27" y="-12.446" size="1.778" layer="51" font="vector">Revised By: Elias Santistevan</text>
-<dimension x1="0" y1="25.4" x2="25.4" y2="25.4" x3="12.7" y3="29.21" textsize="1.778" textratio="15" layer="47" dtype="horizontal" unit="inch"/>
-<dimension x1="25.4" y1="25.4" x2="25.4" y2="0" x3="30.48" y3="12.7" textsize="1.778" textratio="15" layer="47" dtype="horizontal" unit="inch"/>
-<text x="3.81" y="34.29" size="1.778" layer="47" font="vector" ratio="15">Units in Inches</text>
+<text x="32.131" y="-20.066" size="1.778" layer="51" font="vector" align="bottom-right">Michelle Shorter</text>
+<text x="-2.286" y="-22.86" size="1.778" layer="51" font="vector">Revised By: Elias Santistevan</text>
 <circle x="18.034" y="11.176" radius="0.643075" width="0.3048" layer="21"/>
 <circle x="18.034" y="11.176" radius="0.6604" width="0.3048" layer="22"/>
+<dimension x1="2.54" y1="2.54" x2="22.86" y2="2.54" x3="12.7" y3="-3.048" textsize="1.778" textratio="15" layer="47" unit="inch"/>
+<dimension x1="25.4" y1="0" x2="0" y2="0" x3="12.7" y3="-6.35" textsize="1.778" textratio="15" layer="47" dtype="horizontal" unit="inch"/>
+<dimension x1="22.86" y1="22.86" x2="22.86" y2="2.54" x3="28.702" y3="12.7" textsize="1.778" textratio="15" layer="47" unit="inch"/>
+<dimension x1="25.4" y1="25.4" x2="25.4" y2="0" x3="33.274" y3="12.7" textsize="1.778" textratio="15" layer="47" unit="inch"/>
+<text x="4.064" y="-9.398" size="1.778" layer="47" font="vector" ratio="15">Units in Inches</text>
 </plain>
 <attributes>
@@
 <attribute name="VALUE" x="26.162" y="15.24" size="0.6096" layer="27" font="vector" ratio="20" rot="R90"/>
 </element>
-<element name="FRAME1" library="SparkFun-Aesthetics" package="CREATIVE_COMMONS" value="FRAME-LETTER" x="-10.16" y="-9.652" smashed="yes">
-<attribute name="DESIGNER" value="" x="-10.16" y="-9.652" size="1.778" layer="27" font="vector" ratio="15" display="off"/>
-<attribute name="REV" value="" x="-10.16" y="-9.652" size="1.778" layer="27" font="vector" ratio="15" display="off"/>
+<element name="FRAME1" library="SparkFun-Aesthetics" package="CREATIVE_COMMONS" value="FRAME-LETTER" x="-13.716" y="-20.066" smashed="yes">
+<attribute name="DESIGNER" value="" x="-13.716" y="-20.066" size="1.778" layer="27" font="vector" ratio="15" display="off"/>
+<attribute name="REV" value="" x="-13.716" y="-20.066" size="1.778" layer="27" font="vector" ratio="15" display="off"/>
 </element>
 <element name="LOGO3" library="SparkFun-Aesthetics" package="OSHW-LOGO-S" value="OSHW-LOGOS" x="16.256" y="18.034" smashed="yes" rot="MR0"/>
@@
 <element name="LOGO1" library="SparkFun-Aesthetics" package="SFE_LOGO_NAME_.1" value="SFE_LOGO_NAME.1_INCH" x="13.208" y="7.62" smashed="yes" rot="MR0"/>
 <element name="TP1" library="SparkFun-Connectors" package="TP_15TH" value="TEST-POINTTP_15TH_THRU" x="16.8402" y="20.4978" smashed="yes"/>
-<element name="J2" library="SparkFun-Connectors" package="1X04_NO_SILK" value="" x="24.13" y="6.604" smashed="yes" rot="R90">
-<attribute name="NAME" x="22.733" y="5.334" size="0.6096" layer="25" font="vector" ratio="20" rot="R90"/>
-<attribute name="PROD_ID" value="CONN-09696" x="24.13" y="6.604" size="1.778" layer="27" rot="R90" display="off"/>
-<attribute name="VALUE" x="26.162" y="5.334" size="0.6096" layer="27" font="vector" ratio="20" rot="R90"/>
+<element name="J2" library="SparkFun-Connectors" package="1X04_NO_SILK" value="" x="24.13" y="6.35" smashed="yes" rot="R90">
+<attribute name="NAME" x="22.733" y="5.08" size="0.6096" layer="25" font="vector" ratio="20" rot="R90"/>
+<attribute name="PROD_ID" value="CONN-09696" x="24.13" y="6.35" size="1.778" layer="27" rot="R90" display="off"/>
+<attribute name="VALUE" x="26.162" y="5.08" size="0.6096" layer="27" font="vector" ratio="20" rot="R90"/>
 </element>
 <element name="FD2" library="SparkFun-Aesthetics" package="FIDUCIAL-MICRO" value="FIDUCIALUFIDUCIAL" x="0.762" y="0.762" smashed="yes"/>
@@
 <contactref element="J2" pad="4"/>
 <wire x1="22.5679" y1="12.4079" x2="24.13" y2="13.97" width="0.2032" layer="16"/>
-<wire x1="24.13" y1="13.97" x2="24.13" y2="14.224" width="0.2032" layer="16"/>
 <contactref element="U3" pad="PA09"/>
 <wire x1="12.1264" y1="11.14" x2="10.01" y2="11.14" width="0.2032" layer="1"/>
@@
 <wire x1="13.2" y1="9.5076" x2="12.0676" y2="10.64" width="0.2032" layer="1"/>
 <contactref element="J2" pad="3"/>
-<wire x1="24.13" y1="11.684" x2="24.13" y2="11.176" width="0.2032" layer="16"/>
+<wire x1="24.13" y1="11.43" x2="24.13" y2="11.176" width="0.2032" layer="16"/>
 <wire x1="13.2" y1="5.08" x2="13.2" y2="7.112" width="0.2032" layer="1"/>
 <contactref element="U3" pad="PA08"/>
@@
 <wire x1="4.6176" y1="10.6934" x2="4.318" y2="10.6934" width="0.254" layer="1"/>
 <contactref element="J2" pad="2"/>
-<wire x1="23.1013" y1="8.6233" x2="23.622" y2="9.144" width="0.254" layer="16"/>
-<wire x1="23.622" y1="9.144" x2="24.13" y2="9.144" width="0.254" layer="16"/>
+<wire x1="23.1013" y1="8.6233" x2="23.368" y2="8.89" width="0.254" layer="16"/>
+<wire x1="23.368" y1="8.89" x2="24.13" y2="8.89" width="0.254" layer="16"/>
 <contactref element="U2" pad="3"/>
 <contactref element="R2" pad="2"/>

Commit message: Swaps "D16/D17" symbol names
Parts:
- J1: value (none) -> QWIIC_RIGHT_ANGLE
Changed lines of the file:
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@@
 <?xml version="1.0" encoding="utf-8"?>
 <!DOCTYPE eagle SYSTEM "eagle.dtd">
-<eagle version="9.4.2">
+<eagle version="9.6.2">
 <drawing>
 <settings>
@@
 <setting verticaltext="up"/>
 </settings>
-<grid distance="0.01" unitdist="inch" unit="inch" style="lines" multiple="1" display="yes" altdistance="0.001" altunitdist="inch" altunit="inch"/>
+<grid distance="0.05" unitdist="inch" unit="inch" style="dots" multiple="1" display="yes" altdistance="0.005" altunitdist="inch" altunit="inch"/>
 <layers>
 <layer number="1" name="Top" color="4" fill="1" visible="yes" active="yes"/>
 <layer number="2" name="Route2" color="1" fill="3" visible="no" active="yes"/>
 <layer number="15" name="Route15" color="4" fill="6" visible="no" active="yes"/>
-<layer number="16" name="Bottom" color="31" fill="1" visible="yes" active="yes"/>
-<layer number="17" name="Pads" color="30" fill="1" visible="yes" active="yes"/>
+<layer number="16" name="Bottom" color="3" fill="1" visible="yes" active="yes"/>
+<layer number="17" name="Pads" color="26" fill="1" visible="yes" active="yes"/>
 <layer number="18" name="Vias" color="2" fill="1" visible="yes" active="yes"/>
 <layer number="19" name="Unrouted" color="6" fill="1" visible="yes" active="yes"/>
@@
 <layer number="115" name="ReferenceISLANDS" color="7" fill="1" visible="no" active="no"/>
 <layer number="116" name="Patch_BOT" color="9" fill="4" visible="no" active="no"/>
-<layer number="117" name="PM_Ref" color="26" fill="1" visible="no" active="yes"/>
+<layer number="117" name="PM_Ref" color="26" fill="1" visible="yes" active="yes"/>
 <layer number="118" name="Rect_Pads" color="7" fill="1" visible="no" active="no"/>
-<layer number="119" name="PF_Ref" color="31" fill="1" visible="no" active="yes"/>
-<layer number="120" name="WFL_Ref" color="25" fill="1" visible="no" active="yes"/>
+<layer number="119" name="PF_Ref" color="31" fill="1" visible="yes" active="yes"/>
+<layer number="120" name="WFL_Ref" color="25" fill="1" visible="yes" active="yes"/>
 <layer number="121" name="_tsilk" color="7" fill="1" visible="no" active="no"/>
 <layer number="122" name="_bsilk" color="7" fill="1" visible="no" active="no"/>
@@
 <layer number="128" name="_bValues" color="7" fill="1" visible="no" active="no"/>
 <layer number="129" name="Mask" color="7" fill="1" visible="no" active="no"/>
+<layer number="130" name="SMDSTROOK" color="7" fill="1" visible="no" active="no"/>
 <layer number="131" name="tAdjust" color="7" fill="1" visible="no" active="no"/>
 <layer number="132" name="bAdjust" color="7" fill="1" visible="no" active="no"/>
+<layer number="133" name="bottom_silk" color="7" fill="1" visible="no" active="no"/>
+<layer number="134" name="silk_top" color="7" fill="1" visible="no" active="no"/>
+<layer number="135" name="silk_bottom" color="7" fill="1" visible="no" active="no"/>
+<layer number="136" name="silktop" color="7" fill="1" visible="no" active="no"/>
+<layer number="137" name="silkbottom" color="7" fill="1" visible="no" active="no"/>
+<layer number="138" name="EEE" color="7" fill="1" visible="no" active="no"/>
+<layer number="139" name="_tKeepout" color="7" fill="1" visible="no" active="no"/>
+<layer number="140" name="mbKeepout" color="7" fill="1" visible="no" active="no"/>
+<layer number="141" name="ASSEMBLY_TOP" color="7" fill="1" visible="no" active="no"/>
+<layer number="142" name="mbRestrict" color="7" fill="1" visible="no" active="no"/>
+<layer number="143" name="PLACE_BOUND_TOP" color="7" fill="1" visible="no" active="no"/>
 <layer number="144" name="Drill_legend" color="7" fill="1" visible="no" active="no"/>
+<layer number="145" name="DrillLegend_01-16" color="7" fill="1" visible="no" active="no"/>
+<layer number="146" name="DrillLegend_01-20" color="7" fill="1" visible="no" active="no"/>
+<layer number="147" name="PIN_NUMBER" color="7" fill="1" visible="no" active="no"/>
+<layer number="148" name="DrillLegend_01-20" color="7" fill="1" visible="no" active="no"/>
+<layer number="149" name="DrillLegend_02-15" color="7" fill="1" visible="no" active="no"/>
 <layer number="150" name="Notes" color="7" fill="1" visible="no" active="no"/>
 <layer number="151" name="HeatSink" color="7" fill="1" visible="no" active="no"/>
@@
 <layer number="154" name="FabDoc2" color="7" fill="1" visible="no" active="no"/>
 <layer number="155" name="FabDoc3" color="7" fill="1" visible="no" active="no"/>
+<layer number="166" name="AntennaArea" color="7" fill="1" visible="no" active="no"/>
+<layer number="168" name="4mmHeightArea" color="7" fill="1" visible="no" active="no"/>
+<layer number="191" name="mNets" color="7" fill="1" visible="no" active="no"/>
+<layer number="192" name="mBusses" color="7" fill="1" visible="no" active="no"/>
+<layer number="193" name="mPins" color="7" fill="1" visible="no" active="no"/>
+<layer number="194" name="mSymbols" color="7" fill="1" visible="no" active="no"/>
+<layer number="195" name="mNames" color="7" fill="1" visible="no" active="no"/>
+<layer number="196" name="mValues" color="7" fill="1" visible="no" active="no"/>
 <layer number="199" name="Contour" color="7" fill="1" visible="no" active="no"/>
 <layer number="200" name="200bmp" color="1" fill="10" visible="no" active="no"/>
@@
 </autorouter>
 <elements>
-<element name="J1" library="SparkFun-Connectors" package="JST04_1MM_RA" value="" x="12.7" y="5.08" smashed="yes">
+<element name="J1" library="SparkFun-Connectors" package="JST04_1MM_RA" value="QWIIC_RIGHT_ANGLE" x="12.7" y="5.08" smashed="yes">
 <attribute name="NAME" x="11.303" y="2.921" size="0.6096" layer="25" font="vector" ratio="20"/>
 <attribute name="PROD_ID" value="CONN-13694" x="12.7" y="5.08" size="1.778" layer="27" display="off"/>
-<attribute name="VALUE" x="11.049" y="1.778" size="0.6096" layer="27" font="vector" ratio="20"/>
+<attribute name="VALUE" value="QWIIC_RIGHT_ANGLE" x="11.049" y="1.778" size="0.6096" layer="27" font="vector" ratio="20"/>
 </element>
 <element name="J5" library="SparkFun-Connectors" package="USB-MICROB-PTH-MILL" value="" x="6.985" y="20.701" smashed="yes" rot="R180">
@@
 <element name="S2" library="SparkFun-Switches" package="TACTILE_SWITCH_SMD_4.6X2.8MM" value="MOMENTARY-SWITCH-SPST-SMD-4.6X2.8MM" x="20.2438" y="15.494" smashed="yes" rot="R90">
 <attribute name="NAME" x="18.7198" y="15.494" size="0.6096" layer="25" font="vector" ratio="20" rot="R90" align="bottom-center"/>
-<attribute name="PROD_ID" value="SWCH-13065" x="20.2438" y="15.494" size="1.778" layer="27" rot="R90" display="off"/>
+<attribute name="PROD_ID" value="SWCH-15606" x="20.2438" y="15.494" size="1.778" layer="27" rot="R90" display="off"/>
 <attribute name="VALUE" x="21.7678" y="15.494" size="0.6096" layer="27" font="vector" ratio="20" rot="R90" align="top-center"/>
 </element>
@@
 <attribute name="VALUE" x="11.624" y="8.928" size="1" layer="27" rot="R90"/>
 </element>
-<element name="JP1" library="SparkFun-Jumpers" package="SMT-JUMPER_2_NC_TRACE_SILK" value="LED" x="18.288" y="2.032" smashed="yes" rot="MR90">
+<element name="JP1" library="SparkFun-Jumpers" package="SMT-JUMPER_2_NC_TRACE_SILK" package3d_urn="urn:adsk.eagle:package:39281/1" value="LED" x="18.288" y="2.032" smashed="yes" rot="MR90">
 <attribute name="NAME" x="19.431" y="2.032" size="0.6096" layer="26" font="vector" ratio="20" rot="MR90" align="bottom-center"/>
 <attribute name="VALUE" x="17.145" y="2.032" size="0.6096" layer="28" font="vector" ratio="20" rot="MR90" align="top-center"/>
@@
 <contactref element="JP1" pad="2"/>
 <wire x1="15.24" y1="3.81" x2="16.51" y2="2.54" width="0.254" layer="16"/>
-<wire x1="16.51" y1="2.54" x2="18.288" y2="2.54" width="0.254" layer="16"/>
+<wire x1="16.51" y1="2.54" x2="18.288" y2="2.5527" width="0.254" layer="16"/>
 <wire x1="20.6248" y1="12.6492" x2="18.2922" y2="12.6492" width="0.254" layer="1"/>
 <wire x1="18.2922" y1="12.6492" x2="18.034" y2="12.9074" width="0.254" layer="1"/>
@@
 <wire x1="18.741" y1="0.9652" x2="18.7918" y2="0.9144" width="0.2032" layer="1"/>
 <wire x1="19.7612" y1="0.9144" x2="18.8976" y2="0.9144" width="0.2032" layer="16"/>
-<wire x1="18.8976" y1="0.9144" x2="18.288" y2="1.524" width="0.2032" layer="16"/>
+<wire x1="18.8976" y1="0.9144" x2="18.288" y2="1.5113" width="0.2032" layer="16"/>
 </signal>
 <signal name="N$4">
@@
 </board>
 </drawing>
+<compatibility>
+<note version="8.3" severity="warning">
+Since Version 8.3, EAGLE supports URNs for individual library
+assets (packages, symbols, and devices). The URNs of those assets
+will not be understood (or retained) with this version.
+</note>
+<note version="8.3" severity="warning">
+Since Version 8.3, EAGLE supports the association of 3D packages
+with devices in libraries, schematics, and board files. Those 3D
+packages will not be understood (or retained) with this version.
+</note>
+</compatibility>
 </eagle>
